File: output/pcbs/tutorial.kicad_pcb (KiCad board)
At the start: 2 copper layers, 136 x 102.2 mm, 66 parts

Commit message: pcb changes
Parts:
- moved MCU1 109.6 mm to (152.9, 52.7)
- moved D1 108.2 mm to (42.5, 104.5)
- moved D10 108.2 mm to (78.5, 81.5)
- moved D11 108.2 mm to (78.5, 64.5)
- moved D12 108.2 mm to (78.5, 47.5)
- moved D13 108.2 mm to (96.5, 97.0)
- moved D14 108.2 mm to (96.5, 80.0)
- moved D15 108.2 mm to (96.5, 63.0)
- moved D16 108.2 mm to (96.5, 46.0)
- moved D17 108.2 mm to (114.5, 99.0)
- moved D18 108.2 mm to (114.5, 82.0)
- moved D19 108.2 mm to (114.5, 65.0)
- moved D2 108.2 mm to (42.5, 87.5)
- moved D20 108.2 mm to (114.5, 48.0)
- moved D21 108.2 mm to (132.5, 101.0)
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Routing:
- net P3: track 0.00 -> 247.5 mm, vias 0 -> 6
- net P4: track 0.00 -> 199.6 mm, vias 0 -> 6
- net P2: track 0.00 -> 197.6 mm, vias 0 -> 5
- net P16: track 0.00 -> 187.7 mm, vias 0 -> 1
- net P6: track 0.00 -> 184.7 mm, vias 0 -> 5
- net P5: track 0.00 -> 173.2 mm, vias 0 -> 5
- net P14: track 0.00 -> 159.0 mm, vias 0 -> 1
- net P15: track 0.00 -> 153.3 mm
- net P18: track 0.00 -> 152.7 mm
- net P7: track 0.00 -> 105.1 mm, vias 0 -> 4
- net GND: track 0.00 -> 72.9 mm
- net P10: track 0.00 -> 67.9 mm
- net D10: track 0.00 -> 50.2 mm
- net ring_bottom: track 0.00 -> 35.0 mm
- net thumb_hey: track 0.00 -> 32.7 mm
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Other:
- net class Default removed
